File: STM32F303-RIR4.kicad_sch (KiCad schematic)
At the start: 34 parts, among them J0 CN7, J1 CN10, J101 LCC, J102 LCC, J103 S4 S3 S2 S1 SC, J104 MA MB NA NB, J105 - 12V +, J106 Servo 4, J107 Servo 3, J108 Servo 2, J109 Servo 1, J110 B1 C B2, U101 SN65HVD1050, U102 LM358, U103 TBD62064AFG, U104 TC4428, U105 TC4428, U106 G3VM-61VY4, U107 G3VM-61VY4

Commit message: Assorted minor updates.
Parts:
- C101: Mouser Part Number (none) -> 963-EMK107B7104KAHT
- U101: Mouser Part Number (none) -> 595-SN65HVD1050DR
- U103: footprint SOP100P800X190:SOP100P800X190-24N -> MyHSOP:HSOP16-P-300-1.00; Mouser Part Number (none) -> 757-TBD62064AFGEL
Connections:
- net +12V: now also U103.8 (OC), U103.8 (OC), U103.8 (OC), U103.8 (OC); no longer U103.12 (OC)
- net GND: now also U103.FIN (GND), U103.FIN (GND), U103.FIN (GND), U103.FIN (GND); no longer U103.17 (GND), U103.18 (GND), U103.19 (GND), U103.20 (GND), U103.5 (GND), U103.6 (GND), U103.7 (GND), U103.8 (GND)
- net at J0.13 (PA13): now also U103.11 (In); no longer U103.15 (In)
- net at J0.15 (PA14): now also U103.14 (In); no longer U103.22 (In)
- net at J0.3 (PC12): now also U103.6 (In); no longer U103.10 (In)
- net at J103.3 (Pin_3): now also U103.7 (Out); no longer U103.11 (Out)
- net at J103.4 (Pin_4): now also U103.9 (Out); no longer U103.13 (Out)
- net at J103.5 (Pin_5): now also U103.13 (Out); no longer U103.24 (Out)

Commit message: Finalize part numbers.
Parts:
- R107, R108: Mouser Part Number (none) -> 603-RE0603FRE07330RL
- U104, U105: Mouser Part Number (none) -> 579-TC1428COA
Changed lines of the file:
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@@
       (effects (font (size 1.524 1.524)))
+    )
+    (property "Mouser Part Number" "579-TC1428COA" (id 4) (at 45.085 104.14 0)
+      (effects (font (size 1.27 1.27)) hide)
     )
     (pin "3")
@@
       (effects (font (size 1.524 1.524)))
     )
+    (property "Mouser Part Number" "579-TC1428COA" (id 4) (at 45.085 125.73 0)
+      (effects (font (size 1.27 1.27)) hide)
+    )
     (pin "3")
     (pin "6")
@@
       (effects (font (size 1.524 1.524)))
     )
+    (property "Mouser Part Number" "579-TC1428COA" (id 4) (at 44.45 144.78 0)
+      (effects (font (size 1.27 1.27)) hide)
+    )
     (pin "3")
     (pin "6")
@@
     (property "Datasheet" "" (id 3) (at 44.45 167.005 0)
       (effects (font (size 1.524 1.524)))
+    )
+    (property "Mouser Part Number" "579-TC1428COA" (id 4) (at 44.45 167.005 0)
+      (effects (font (size 1.27 1.27)) hide)
     )
     (pin "3")
@@
       (effects (font (size 1.27 1.27)) hide)
     )
+    (property "Mouser Part Number" "603-RE0603FRE07330RL" (id 4) (at 146.05 97.155 90)
+      (effects (font (size 1.27 1.27)) hide)
+    )
     (pin "1")
     (pin "2")
@@
       (effects (font (size 1.27 1.27)) hide)
     )
+    (property "Mouser Part Number" "603-RE0603FRE07330RL" (id 4) (at 146.05 111.76 90)
+      (effects (font (size 1.27 1.27)) hide)
+    )

Commit message: Prep for PCB making.
Parts:
- C101: LCSC (none) -> C2173920; MPN (none) -> Taiyo Yuden EMK107B7104KAHT
- D101: LCSC (none) -> C7083723; MPN (none) -> Lumex SML-LX0603YW-TR
- D102: LCSC (none) -> C5354817; MPN (none) -> Lumex SML-LX0603IW-TR
- R101, R102: LCSC (none) -> C228185; MPN (none) -> YAGEO AC0603JR-07390RL
- R107, R108: LCSC (none) -> C859411; MPN (none) -> YAGEO RE0603FRE07330RL
- U101: LCSC (none) -> C14019; MPN (none) -> TI SN65HVD1050DR
- U102: LCSC (none) -> C5145450; MPN (none) -> HANSCHIP semiconductor LM358DRG
- U103: LCSC (none) -> C141521; MPN (none) -> TOSHIBA TBD62064AFG,EL
- U104, U105: LCSC (none) -> C636863; MPN (none) -> MICROCHIP TC1428COA
- U106, U107: LCSC (none) -> C19844354; MPN (none) -> OMRON G3VM-61VY4(TR05)
Changed lines of the file:
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@@
+      (effects (font (size 1.27 1.27)) hide)
+    )
+    (property "LCSC" "C14019" (id 5) (at 194.31 130.175 0)
+      (effects (font (size 1.27 1.27)) hide)
+    )
+    (property "MPN" "TI SN65HVD1050DR" (id 6) (at 194.31 130.175 0)
       (effects (font (size 1.27 1.27)) hide)
     )
@@
       (effects (font (size 1.27 1.27)) hide)
     )
+    (property "LCSC" "C2173920" (id 5) (at 206.375 121.285 0)
+      (effects (font (size 1.27 1.27)) hide)
+    )
+    (property "MPN" "Taiyo Yuden EMK107B7104KAHT" (id 6) (at 206.375 121.285 0)
+      (effects (font (size 1.27 1.27)) hide)
+    )
     (pin "1")
     (pin "2")
@@
       (effects (font (size 1.524 1.524)) hide)
     )
+    (property "LCSC" "C5145450" (id 5) (at 193.04 78.74 0)
+      (effects (font (size 1.27 1.27)) hide)
+    )
+    (property "MPN" "HANSCHIP semiconductor LM358DRG" (id 6) (at 193.04 78.74 0)
+      (effects (font (size 1.27 1.27)) hide)
+    )
     (pin "4")
     (pin "8")
@@
       (effects (font (size 1.524 1.524)) hide)
     )
+    (property "LCSC" "C5145450" (id 5) (at 193.675 102.235 0)
+      (effects (font (size 1.27 1.27)) hide)
+    )
+    (property "MPN" "HANSCHIP semiconductor LM358DRG" (id 6) (at 193.675 102.235 0)
+      (effects (font (size 1.27 1.27)) hide)
+    )
     (pin "4")
     (pin "8")
@@
       (effects (font (size 1.524 1.524)) hide)
     )
+    (property "LCSC" "C228185" (id 5) (at 210.82 78.74 90)
+      (effects (font (size 1.27 1.27)) hide)
+    )
+    (property "MPN" "YAGEO AC0603JR-07390RL" (id 6) (at 210.82 78.74 90)
+      (effects (font (size 1.27 1.27)) hide)
+    )
     (pin "1")
     (pin "2")
@@
       (effects (font (size 1.524 1.524)) hide)
     )
+    (property "LCSC" "C228185" (id 5) (at 210.185 102.235 90)
+      (effects (font (size 1.27 1.27)) hide)
+    )
+    (property "MPN" "YAGEO AC0603JR-07390RL" (id 6) (at 210.185 102.235 90)
+      (effects (font (size 1.27 1.27)) hide)
+    )
     (pin "1")
     (pin "2")
@@
       (effects (font (size 1.524 1.524)) hide)
     )
+    (property "LCSC" "C7083723" (id 5) (at 213.995 94.615 0)
+      (effects (font (size 1.27 1.27)) hide)
+    )
+    (property "MPN" "Lumex SML-LX0603YW-TR" (id 6) (at 213.995 94.615 0)
+      (effects (font (size 1.27 1.27)) hide)
+    )
     (pin "1")
     (pin "2")
@@
       (effects (font (size 1.524 1.524)) hide)
     )
+    (property "LCSC" "C5354817" (id 5) (at 215.265 70.485 0)
+      (effects (font (size 1.27 1.27)) hide)
+    )
+    (property "MPN" "Lumex SML-LX0603IW-TR" (id 6) (at 215.265 70.485 0)
+      (effects (font (size 1.27 1.27)) hide)
+    )
     (pin "1")
     (pin "2")
@@
     )
     (property "Mouser Part Number" "757-TBD62064AFGEL " (id 4) (at 40.64 43.815 0)
+      (effects (font (size 1.27 1.27)) hide)
+    )
+    (property "LCSC" "C141521" (id 5) (at 41.275 39.37 0)
+      (effects (font (size 1.27 1.27)) hide)
+    )
+    (property "MPN" "TOSHIBA TBD62064AFG,EL" (id 6) (at 41.275 39.37 0)
       (effects (font (size 1.27 1.27)) hide)
     )
@@
       (effects (font (size 1.27 1.27)) hide)
     )
+    (property "LCSC" "C636863" (id 5) (at 45.085 104.14 0)
+      (effects (font (size 1.27 1.27)) hide)
+    )
+    (property "MPN" "MICROCHIP TC1428COA" (id 6) (at 45.085 104.14 0)
+      (effects (font (size 1.27 1.27)) hide)
+    )
     (pin "3")
     (pin "6")
@@
       (effects (font (size 1.27 1.27)) hide)
     )
+    (property "LCSC" "C636863" (id 5) (at 45.085 125.73 0)
+      (effects (font (size 1.27 1.27)) hide)
+    )
+    (property "MPN" "MICROCHIP TC1428COA" (id 6) (at 45.085 125.73 0)
+      (effects (font (size 1.27 1.27)) hide)
+    )
     (pin "3")
     (pin "6")
@@
       (effects (font (size 1.27 1.27)) hide)
     )
+    (property "LCSC" "C636863" (id 5) (at 44.45 144.78 0)
+      (effects (font (size 1.27 1.27)) hide)
+    )
+    (property "MPN" "MICROCHIP TC1428COA" (id 6) (at 44.45 144.78 0)
+      (effects (font (size 1.27 1.27)) hide)
+    )
     (pin "3")
     (pin "6")
@@
       (effects (font (size 1.27 1.27)) hide)
     )
+    (property "LCSC" "C636863" (id 5) (at 44.45 167.005 0)
+      (effects (font (size 1.27 1.27)) hide)
+    )
+    (property "MPN" "MICROCHIP TC1428COA" (id 6) (at 44.45 167.005 0)
+      (effects (font (size 1.27 1.27)) hide)
+    )
     (pin "3")
     (pin "6")
@@
       (effects (font (size 1.524 1.524)) hide)
     )
+    (property "LCSC" "C19844354" (id 5) (at 161.925 99.695 0)
+      (effects (font (size 1.27 1.27)) hide)
+    )
+    (property "MPN" "OMRON G3VM-61VY4(TR05)" (id 6) (at 161.925 99.695 0)
+      (effects (font (size 1.27 1.27)) hide)
+    )
     (pin "1")
     (pin "2")
@@
     (property "Mouser Part Number" " 653-G3VM-61VY4-TR05" (id 4) (at 161.925 114.3 0)
       (effects (font (size 1.524 1.524)) hide)
+    )
+    (property "LCSC" "C19844354" (id 5) (at 161.925 114.3 0)
+      (effects (font (size 1.27 1.27)) hide)
+    )
+    (property "MPN" "OMRON G3VM-61VY4(TR05)" (id 6) (at 161.925 114.3 0)
+      (effects (font (size 1.27 1.27)) hide)
     )
     (pin "1")
@@
       (effects (font (size 1.27 1.27)) hide)
     )
+    (property "LCSC" "C859411" (id 5) (at 146.05 97.155 90)
+      (effects (font (size 1.27 1.27)) hide)
+    )
+    (property "MPN" "YAGEO RE0603FRE07330RL" (id 6) (at 146.05 97.155 90)
+      (effects (font (size 1.27 1.27)) hide)
+    )
     (pin "1")
     (pin "2")
@@
       (effects (font (size 1.27 1.27)) hide)
     )
+    (property "LCSC" "C859411" (id 5) (at 146.05 111.76 90)
+      (effects (font (size 1.27 1.27)) hide)
+    )
+    (property "MPN" "YAGEO RE0603FRE07330RL" (id 6) (at 146.05 111.76 90)
+      (effects (font (size 1.27 1.27)) hide)
+    )
     (pin "1")
     (pin "2")
@@
     )
     (property "Mouser Part Number" "757-TBD62064AFGEL " (id 4) (at 40.64 55.245 0)
+      (effects (font (size 1.27 1.27)) hide)
+    )
+    (property "LCSC" "C141521" (id 5) (at 41.275 50.8 0)
+      (effects (font (size 1.27 1.27)) hide)
+    )
+    (property "MPN" "TOSHIBA TBD62064AFG,EL" (id 6) (at 41.275 50.8 0)
       (effects (font (size 1.27 1.27)) hide)
     )
@@
       (effects (font (size 1.27 1.27)) hide)
     )
+    (property "LCSC" "C141521" (id 5) (at 41.275 63.5 0)
+      (effects (font (size 1.27 1.27)) hide)
+    )
+    (property "MPN" "TOSHIBA TBD62064AFG,EL" (id 6) (at 41.275 63.5 0)
+      (effects (font (size 1.27 1.27)) hide)
+    )
     (pin "1")
     (pin "8")
@@
       (effects (font (size 1.27 1.27)) hide)
     )
+    (property "LCSC" "C141521" (id 5) (at 41.275 78.74 0)
+      (effects (font (size 1.27 1.27)) hide)
+    )
+    (property "MPN" "TOSHIBA TBD62064AFG,EL" (id 6) (at 41.275 78.74 0)
+      (effects (font (size 1.27 1.27)) hide)
+    )

Commit message: Prep for PCB making.
Parts:
- J0, J1, J101, J102, J103, J104, J105, J106, J107, J108, J109, J110, MK101, MK102, MK103, MK104, R103, R104, R105, R106: now left out of the parts list
Changed lines of the file:
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@@
   )
   (symbol (lib_id "stm32Morpho:CN7") (at 94.615 54.61 0) (unit 1)
-    (in_bom yes) (on_board yes)
+    (in_bom no) (on_board yes)
     (property "Reference" "J0" (id 0) (at 95.885 29.21 0))
     (property "Value" "CN7" (id 1) (at 95.885 80.01 0))
@@
   )
   (symbol (lib_id "stm32Morpho:CN10") (at 158.115 55.88 0) (unit 1)
-    (in_bom yes) (on_board yes)
+    (in_bom no) (on_board yes)
     (property "Reference" "J1" (id 0) (at 159.385 30.48 0))
     (property "Value" "CN10" (id 1) (at 159.385 81.28 0))
@@
   )
   (symbol (lib_id "STM32F303-RIR4-rescue:RJ45") (at 236.855 107.95 270) (unit 1)
-    (in_bom yes) (on_board yes)
+    (in_bom no) (on_board yes)
     (property "Reference" "J102" (id 0) (at 249.555 113.03 0))
     (property "Value" "LCC" (id 1) (at 249.555 104.14 0))
@@
   )
   (symbol (lib_id "STM32F303-RIR4-rescue:RJ45") (at 238.125 151.13 270) (unit 1)
-    (in_bom yes) (on_board yes)
+    (in_bom no) (on_board yes)
     (property "Reference" "J101" (id 0) (at 250.825 156.21 0))
     (property "Value" "LCC" (id 1) (at 250.825 147.32 0))
@@
   )
   (symbol (lib_id "STM32F303-RIR4-rescue:Mounting_Hole") (at 175.26 151.765 0) (unit 1)
-    (in_bom yes) (on_board yes)
+    (in_bom no) (on_board yes)
     (property "Reference" "MK101" (id 0) (at 175.26 146.685 0))
     (property "Value" "Mounting_Hole" (id 1) (at 175.26 148.59 0))
@@
   )
   (symbol (lib_id "STM32F303-RIR4-rescue:Mounting_Hole") (at 173.355 142.24 0) (unit 1)
-    (in_bom yes) (on_board yes)
+    (in_bom no) (on_board yes)
     (property "Reference" "MK102" (id 0) (at 173.355 137.16 0))
     (property "Value" "Mounting_Hole" (id 1) (at 173.355 139.065 0))
@@
   )
   (symbol (lib_id "STM32F303-RIR4-rescue:Mounting_Hole") (at 167.005 152.4 0) (unit 1)
-    (in_bom yes) (on_board yes)
+    (in_bom no) (on_board yes)
     (property "Reference" "MK103" (id 0) (at 167.005 147.32 0))
     (property "Value" "Mounting_Hole" (id 1) (at 167.005 149.225 0))
@@
   )
   (symbol (lib_id "STM32F303-RIR4-rescue:Mounting_Hole") (at 163.83 142.24 0) (unit 1)
-    (in_bom yes) (on_board yes)
+    (in_bom no) (on_board yes)
     (property "Reference" "MK104" (id 0) (at 163.83 137.16 0))
     (property "Value" "Mounting_Hole" (id 1) (at 163.83 139.065 0))
@@
   )
   (symbol (lib_id "STM32F303-RIR4-rescue:Screw_Terminal_01x05") (at 19.05 53.975 0) (mirror y) (unit 1)
-    (in_bom yes) (on_board yes)
+    (in_bom no) (on_board yes)
     (property "Reference" "J103" (id 0) (at 19.05 46.355 0))
     (property "Value" "S4 S3 S2 S1 SC" (id 1) (at 19.05 61.595 0))
@@
   )
   (symbol (lib_id "STM32F303-RIR4-rescue:Screw_Terminal_01x04") (at 17.78 133.985 0) (mirror y) (unit 1)
-    (in_bom yes) (on_board yes)
+    (in_bom no) (on_board yes)
     (property "Reference" "J104" (id 0) (at 17.78 128.905 0))
     (property "Value" "MA MB NA NB" (id 1) (at 17.78 141.605 0))
@@
   )
   (symbol (lib_id "STM32F303-RIR4-rescue:Screw_Terminal_01x02") (at 19.685 90.805 0) (mirror y) (unit 1)
-    (in_bom yes) (on_board yes)
+    (in_bom no) (on_board yes)
     (property "Reference" "J105" (id 0) (at 19.685 88.265 0))
     (property "Value" "- 12V +" (id 1) (at 19.685 95.885 0))
@@
   )
   (symbol (lib_id "STM32F303-RIR4-rescue:Conn_01x03_Male") (at 201.93 60.96 0) (mirror y) (unit 1)
-    (in_bom yes) (on_board yes)
+    (in_bom no) (on_board yes)
     (property "Reference" "J109" (id 0) (at 201.93 55.88 0))
     (property "Value" "Servo 1" (id 1) (at 201.93 66.04 0))
@@
   )
   (symbol (lib_id "STM32F303-RIR4-rescue:Conn_01x03_Male") (at 201.93 52.07 0) (mirror y) (unit 1)
-    (in_bom yes) (on_board yes)
+    (in_bom no) (on_board yes)
     (property "Reference" "J108" (id 0) (at 201.93 46.99 0))
     (property "Value" "Servo 2" (id 1) (at 201.93 57.15 0))
@@
   )
   (symbol (lib_id "STM32F303-RIR4-rescue:Conn_01x03_Male") (at 201.93 42.545 0) (mirror y) (unit 1)
-    (in_bom yes) (on_board yes)
+    (in_bom no) (on_board yes)
     (property "Reference" "J107" (id 0) (at 201.93 37.465 0))
     (property "Value" "Servo 3" (id 1) (at 201.93 47.625 0))
@@
   )
   (symbol (lib_id "STM32F303-RIR4-rescue:Conn_01x03_Male") (at 201.93 31.115 0) (mirror y) (unit 1)
-    (in_bom yes) (on_board yes)
+    (in_bom no) (on_board yes)
     (property "Reference" "J106" (id 0) (at 201.93 26.035 0))
     (property "Value" "Servo 4" (id 1) (at 201.93 36.195 0))
@@
   )
   (symbol (lib_id "STM32F303-RIR4-rescue:R") (at 187.96 24.765 0) (unit 1)
-    (in_bom yes) (on_board yes)
-    (property "Reference" "R103" (id 0) (at 189.992 24.765 90))
-    (property "Value" "5K to 20K" (id 1) (at 187.96 24.765 90))
+    (in_bom no) (on_board yes)
+    (property "Reference" "R103" (id 0) (at 191.135 24.765 90))
+    (property "Value" "5K to 20K" (id 1) (at 185.42 24.765 90))
     (property "Footprint" "Resistors_THT:R_Axial_DIN0204_L3.6mm_D1.6mm_P7.62mm_Horizontal" (id 2) (at 186.182 24.765 90)
       (effects (font (size 1.27 1.27)) hide)
@@
   )
   (symbol (lib_id "STM32F303-RIR4-rescue:R") (at 187.96 36.195 0) (unit 1)
-    (in_bom yes) (on_board yes)
-    (property "Reference" "R104" (id 0) (at 189.992 36.195 90))
-    (property "Value" "5K to 20K" (id 1) (at 187.96 36.195 90))
+    (in_bom no) (on_board yes)
+    (property "Reference" "R104" (id 0) (at 191.135 36.195 90))
+    (property "Value" "5K to 20K" (id 1) (at 184.785 36.195 90))
     (property "Footprint" "Resistors_THT:R_Axial_DIN0204_L3.6mm_D1.6mm_P7.62mm_Horizontal" (id 2) (at 186.182 36.195 90)
       (effects (font (size 1.27 1.27)) hide)
@@
   )
   (symbol (lib_id "STM32F303-RIR4-rescue:R") (at 187.96 45.72 0) (unit 1)
-    (in_bom yes) (on_board yes)
+    (in_bom no) (on_board yes)
     (property "Reference" "R105" (id 0) (at 189.992 45.72 90))
-    (property "Value" "5K to 20K" (id 1) (at 187.96 45.72 90))
+    (property "Value" "5K to 20K" (id 1) (at 185.42 45.72 90))
     (property "Footprint" "Resistors_THT:R_Axial_DIN0204_L3.6mm_D1.6mm_P7.62mm_Horizontal" (id 2) (at 186.182 45.72 90)
       (effects (font (size 1.27 1.27)) hide)
@@
   )
   (symbol (lib_id "STM32F303-RIR4-rescue:R") (at 187.96 54.61 0) (unit 1)
-    (in_bom yes) (on_board yes)
+    (in_bom no) (on_board yes)
     (property "Reference" "R106" (id 0) (at 189.992 54.61 90))
-    (property "Value" "5K to 20K" (id 1) (at 187.96 54.61 90))
+    (property "Value" "5K to 20K" (id 1) (at 186.055 54.61 90))
     (property "Footprint" "Resistors_THT:R_Axial_DIN0204_L3.6mm_D1.6mm_P7.62mm_Horizontal" (id 2) (at 186.182 54.61 90)
       (effects (font (size 1.27 1.27)) hide)
@@
   )
   (symbol (lib_id "STM32F303-RIR4-rescue:Screw_Terminal_01x03") (at 177.8 106.045 0) (unit 1)
-    (in_bom yes) (on_board yes)
+    (in_bom no) (on_board yes)
     (property "Reference" "J110" (id 0) (at 177.8 100.965 0))
     (property "Value" "B1 C B2" (id 1) (at 177.8 111.125 0))

Commit message: Add Schematic PDF and Top 3D view png.
Other:
- company: (none) -> Deepwoods Software
- title: (none) -> STM32F303-RIR4
Changed lines of the file:
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@@
 (kicad_sch (version 20211123) (generator eeschema)
-  (paper "A4")
+  (paper "USLetter")
+  (title_block
+    (title "STM32F303-RIR4")
+    (date "7/23/2025")
+    (rev "A")
+    (company "Deepwoods Software")
+  )
   (junction (at 171.45 106.045) (diameter 0) (color 0 0 0 0)
   )
